File: extras/hardware/LMP91000.brd (EAGLE design)
At the start: 20.3 x 17.8 mm, 10 parts

Commit message: making some mods
Parts:
- C1: device CalvEngIO-Passives:C0402 -> LinnesLab-Passives:C0402
- J1: device CalvEngIO-Connectors:1X07_NO_SILK -> LinnesLab-Connectors:1X07_NO_SILK
- J4: device CalvEngIO-Connectors:1X05_NO_SILK -> LinnesLab-Connectors:1X05_NO_SILK
- LMP91000: device CalvEngIO-Sensors:WSON-14 -> LinnesLab-Sensors:WSON-14
- LOGO1: device CalvEngIO-Logos:OSHW-LOGO-S -> LinnesLab-Logos:OSHW-LOGO-S
- R1, R2: device CalvEngIO-Passives:R0402 -> LinnesLab-Passives:R0402-BIGGER
- U$1: device CalvEngIO-Logos:LINNES.LAB.05 -> LinnesLab-Logos:LINNES.LAB.05
- U$2: device CalvEngIO-Logos:LINNES.LAB.LOGO -> LinnesLab-Logos:LINNES.LAB.LOGO
- U$3: device CalvEngIO-Symbols:REV.B -> LinnesLab-Logos:REV.B
